Commit message: model by pkg

File: kobuki_description/urdf/kobuki.urdf.xacro (robot description, xacro)
@@ -30,5 +30,5 @@
         <geometry>
           <!-- new mesh -->
-          <mesh filename="model://kobuki_description/meshes/main_body.dae" />
+          <mesh filename="package://kobuki_description/meshes/main_body.dae" />
         </geometry>
         <origin xyz="0.001 0 0.05199" rpy="0 0 0"/>
@@ -65,5 +65,5 @@
       <visual>
         <geometry>
-          <mesh filename="model://kobuki_description/meshes/wheel.dae"/>
+          <mesh filename="package://kobuki_description/meshes/wheel.dae"/>
         </geometry>
         <origin xyz="0 0 0" rpy="0 0 0"/>
@@ -92,5 +92,5 @@
       <visual>
         <geometry>
-          <mesh filename="model://kobuki_description/meshes/wheel.dae"/>
+          <mesh filename="package://kobuki_description/meshes/wheel.dae"/>
         </geometry>
         <origin xyz="0 0 0" rpy="0 0 0"/>
@@ -228,5 +228,5 @@
 		    <origin xyz="0 0 0" rpy="0 0 0"/>
 		    <geometry>
-			    <mesh filename="model://hokuyo/meshes/hokuyo.dae"/>
+			    <mesh filename="package://hokuyo/meshes/hokuyo.dae"/>
 		    </geometry>
 	    </visual>

File: kobuki_description/urdf/sensors/asus_xtion_pro.urdf.xacro (robot description, xacro)
@@ -33,5 +33,5 @@
         <origin xyz="-0.015 0.0035 0.004" rpy="0 0 0"/>
         <geometry>
-          <mesh filename="model://kobuki_description/meshes/sensors/xtion_pro_camera.dae"/>
+          <mesh filename="package://kobuki_description/meshes/sensors/xtion_pro_camera.dae"/>
         </geometry>
       </visual>
@@ -74,5 +74,5 @@
         <origin xyz="0 0 0" rpy="${-M_PI/2} 0 0"/>
         <geometry>
-          <mesh filename="model://kobuki_description/meshes/sensors/xtion_pro_stack.dae"/>
+          <mesh filename="package://kobuki_description/meshes/sensors/xtion_pro_stack.dae"/>
         </geometry>
       </visual>

File: kobuki_description/urdf/sensors/asus_xtion_pro_offset.urdf.xacro (robot description, xacro)
@@ -33,5 +33,5 @@
         <origin xyz="-0.01 0 0" rpy="${-M_PI/2} -${M_PI} ${-M_PI/2}"/>
         <geometry>
-          <mesh filename="model://turtlebot_description/meshes/sensors/asus_xtion_pro_live.dae" scale="${M_SCALE} ${M_SCALE} ${M_SCALE}"/>
+          <mesh filename="package://turtlebot_description/meshes/sensors/asus_xtion_pro_live.dae" scale="${M_SCALE} ${M_SCALE} ${M_SCALE}"/>
         </geometry>
       </visual>

File: kobuki_description/urdf/sensors/kinect.urdf.xacro (robot description, xacro)
@@ -27,5 +27,5 @@
        <origin xyz="0 0 0" rpy="0 0 ${M_PI/2}"/>
         <geometry>
-         <mesh filename="model://turtlebot_description/meshes/sensors/kinect.dae"/>
+         <mesh filename="package://turtlebot_description/meshes/sensors/kinect.dae"/>
         </geometry>
       </visual>

File: kobuki_description/urdf/stacks/circles.urdf.xacro (robot description, xacro)
@@ -18,5 +18,5 @@
         <origin xyz=" 0 0 0 " rpy="0 0 0" />
         <geometry>
-          <mesh filename="model://turtlebot_description/meshes/stacks/circles/68-02403-125_Spacer.dae"/>
+          <mesh filename="package://turtlebot_description/meshes/stacks/circles/68-02403-125_Spacer.dae"/>
         </geometry>
       </visual>
@@ -46,5 +46,5 @@
         <origin xyz=" 0 0 0 " rpy="0 0 0" />
         <geometry>
-          <mesh filename="model://turtlebot_description/meshes/stacks/circles/68-04552-1000-RA_Turtlebot_M-F_Standoff.dae"/>
+          <mesh filename="package://turtlebot_description/meshes/stacks/circles/68-04552-1000-RA_Turtlebot_M-F_Standoff.dae"/>
         </geometry>
       </visual>
@@ -74,5 +74,5 @@
         <origin xyz=" 0 0 0 " rpy="0 0 0" />
         <geometry>
-          <mesh filename="model://turtlebot_description/meshes/stacks/circles/68-04552-2000-RA_Turtlebot_M-F_Standoff.dae"/>
+          <mesh filename="package://turtlebot_description/meshes/stacks/circles/68-04552-2000-RA_Turtlebot_M-F_Standoff.dae"/>
         </geometry>
       </visual>
@@ -102,5 +102,5 @@
         <origin xyz=" 0 0 0 " rpy="0 0 0" />
         <geometry>
-          <mesh filename="model://turtlebot_description/meshes/stacks/circles/68-02421-8000-RA_Turtlebot_F-F_Standoff.dae"/>
+          <mesh filename="package://turtlebot_description/meshes/stacks/circles/68-02421-8000-RA_Turtlebot_F-F_Standoff.dae"/>
         </geometry>
       </visual>
@@ -130,5 +130,5 @@
         <origin xyz=" 0 0 0 " rpy="0 0 0" />
         <geometry>
-          <mesh filename="model://turtlebot_description/meshes/stacks/circles/68-04556-RA_Kinect_Standoff_Assy.dae"/>
+          <mesh filename="package://turtlebot_description/meshes/stacks/circles/68-04556-RA_Kinect_Standoff_Assy.dae"/>
         </geometry>
       </visual>
@@ -162,5 +162,5 @@
         <origin xyz=" 0 0 0 " rpy="0 0 0" />
         <geometry>
-          <mesh filename="model://turtlebot_description/meshes/stacks/circles/plate_0_logo.dae"/>
+          <mesh filename="package://turtlebot_description/meshes/stacks/circles/plate_0_logo.dae"/>
         </geometry>
       </visual>
@@ -192,5 +192,5 @@
         <origin xyz=" 0 0 0 " rpy="0 0 0" />
         <geometry>
-          <mesh filename="model://turtlebot_description/meshes/stacks/circles/plate_1_logo.dae"/>
+          <mesh filename="package://turtlebot_description/meshes/stacks/circles/plate_1_logo.dae"/>
         </geometry>
       </visual>
@@ -222,5 +222,5 @@
         <origin xyz=" 0 0 0 " rpy="0 0 0" />
         <geometry>
-          <mesh filename="model://turtlebot_description/meshes/stacks/circles/plate_1_logo.dae"/>
+          <mesh filename="package://turtlebot_description/meshes/stacks/circles/plate_1_logo.dae"/>
         </geometry>
       </visual>
@@ -254,5 +254,5 @@
         <origin xyz=" 0 0 0 " rpy="0 0 0" />
         <geometry>
-          <mesh filename="model://turtlebot_description/meshes/stacks/circles/plate_2_logo.dae"/>
+          <mesh filename="package://turtlebot_description/meshes/stacks/circles/plate_2_logo.dae"/>
         </geometry>
       </visual>

File: kobuki_description/urdf/stacks/hexagons.urdf.xacro (robot description, xacro)
@@ -19,5 +19,5 @@
         <origin xyz="0 0 0" rpy="0 0 0"/>
         <geometry>
-          <mesh filename="model://kobuki_description/meshes/stacks/hexagons/pole_bottom.dae"/>
+          <mesh filename="package://kobuki_description/meshes/stacks/hexagons/pole_bottom.dae"/>
         </geometry>
       </visual>
@@ -47,5 +47,5 @@
         <origin xyz="0 0 0" rpy="0 ${M_PI} 0"/>
         <geometry>
-          <mesh filename="model://kobuki_description/meshes/stacks/hexagons/pole_middle.dae"/>
+          <mesh filename="package://kobuki_description/meshes/stacks/hexagons/pole_middle.dae"/>
         </geometry>
       </visual>
@@ -75,5 +75,5 @@
         <origin xyz=" 0 0 0" rpy="0 0 0"/>
         <geometry>
-          <mesh filename="model://kobuki_description/meshes/stacks/hexagons/pole_top.dae"/>
+          <mesh filename="package://kobuki_description/meshes/stacks/hexagons/pole_top.dae"/>
         </geometry>
       </visual>
@@ -103,5 +103,5 @@
         <origin xyz="0 0 -0.01" rpy="0 0 0"/>
         <geometry>
-          <mesh filename="model://kobuki_description/meshes/sensors/sensor_pole.dae" />
+          <mesh filename="package://kobuki_description/meshes/sensors/sensor_pole.dae" />
         </geometry>
       </visual>
@@ -142,5 +142,5 @@
         <origin xyz="0 0 0" rpy="0 0 0"/>
         <geometry>
-          <mesh filename="model://kobuki_description/meshes/stacks/hexagons/plate_bottom.dae"/>
+          <mesh filename="package://kobuki_description/meshes/stacks/hexagons/plate_bottom.dae"/>
         </geometry>
       </visual>
@@ -172,5 +172,5 @@
         <origin xyz="0 0 0" rpy="0 0 0"/>
         <geometry>
-          <mesh filename="model://kobuki_description/meshes/stacks/hexagons/plate_middle.dae"/>
+          <mesh filename="package://kobuki_description/meshes/stacks/hexagons/plate_middle.dae"/>
         </geometry>
       </visual>
@@ -204,5 +204,5 @@
         <origin xyz="0 0 0" rpy="0 0 0"/>
         <geometry>
-          <mesh filename="model://kobuki_description/meshes/stacks/hexagons/plate_top.dae"/>
+          <mesh filename="package://kobuki_description/meshes/stacks/hexagons/plate_top.dae"/>
         </geometry>
       </visual>

File: turtlebot_description/urdf/sensors/asus_xtion_pro.urdf.xacro (robot description, xacro)
@@ -33,5 +33,5 @@
         <origin xyz="-0.015 0.0035 0.004" rpy="0 0 0"/>
         <geometry>
-          <mesh filename="model://turtlebot_description/meshes/sensors/xtion_pro_camera.dae"/>
+          <mesh filename="package://turtlebot_description/meshes/sensors/xtion_pro_camera.dae"/>
         </geometry>
       </visual>
@@ -74,5 +74,5 @@
         <origin xyz="0 0 0" rpy="${-M_PI/2} 0 0"/>
         <geometry>
-          <mesh filename="model://turtlebot_description/meshes/sensors/xtion_pro_stack.dae"/>
+          <mesh filename="package://turtlebot_description/meshes/sensors/xtion_pro_stack.dae"/>
         </geometry>
       </visual>

File: turtlebot_description/urdf/stacks/hexagons.urdf.xacro (robot description, xacro)
@@ -19,5 +19,5 @@
         <origin xyz="0 0 0" rpy="0 0 0"/>
         <geometry>
-          <mesh filename="model://turtlebot_description/meshes/stacks/hexagons/pole_bottom.dae"/>
+          <mesh filename="package://turtlebot_description/meshes/stacks/hexagons/pole_bottom.dae"/>
         </geometry>
       </visual>
@@ -47,5 +47,5 @@
         <origin xyz="0 0 0" rpy="0 ${M_PI} 0"/>
         <geometry>
-          <mesh filename="model://turtlebot_description/meshes/stacks/hexagons/pole_middle.dae"/>
+          <mesh filename="package://turtlebot_description/meshes/stacks/hexagons/pole_middle.dae"/>
         </geometry>
       </visual>
@@ -75,5 +75,5 @@
         <origin xyz=" 0 0 0" rpy="0 0 0"/>
         <geometry>
-          <mesh filename="model://turtlebot_description/meshes/stacks/hexagons/pole_top.dae"/>
+          <mesh filename="package://turtlebot_description/meshes/stacks/hexagons/pole_top.dae"/>
         </geometry>
       </visual>
@@ -103,5 +103,5 @@
         <origin xyz="0 0 -0.01" rpy="0 0 0"/>
         <geometry>
-          <mesh filename="model://turtlebot_description/meshes/sensors/sensor_pole.dae" />
+          <mesh filename="package://turtlebot_description/meshes/sensors/sensor_pole.dae" />
         </geometry>
       </visual>
@@ -142,5 +142,5 @@
         <origin xyz="0 0 0" rpy="0 0 0"/>
         <geometry>
-          <mesh filename="model://turtlebot_description/meshes/stacks/hexagons/plate_bottom.dae"/>
+          <mesh filename="package://turtlebot_description/meshes/stacks/hexagons/plate_bottom.dae"/>
         </geometry>
       </visual>
@@ -172,5 +172,5 @@
         <origin xyz="0 0 0" rpy="0 0 0"/>
         <geometry>
-          <mesh filename="model://turtlebot_description/meshes/stacks/hexagons/plate_middle.dae"/>
+          <mesh filename="package://turtlebot_description/meshes/stacks/hexagons/plate_middle.dae"/>
         </geometry>
       </visual>
@@ -204,5 +204,5 @@
         <origin xyz="0 0 0" rpy="0 0 0"/>
         <geometry>
-          <mesh filename="model://turtlebot_description/meshes/stacks/hexagons/plate_top.dae"/>
+          <mesh filename="package://turtlebot_description/meshes/stacks/hexagons/plate_top.dae"/>
         </geometry>
       </visual>

Commit message: Added some changes to kinetic branch

File: kobuki_description/urdf/kobuki.urdf.xacro (robot description, xacro)
@@ -228,5 +228,5 @@
 		    <origin xyz="0 0 0" rpy="0 0 0"/>
 		    <geometry>
-			    <mesh filename="package://hokuyo/meshes/hokuyo.dae"/>
+			    <mesh filename="package://gazebo_plugins/test/multi_robot_scenario/meshes/laser/hokuyo.dae"/>
 		    </geometry>
 	    </visual>
